File: nukeanal.kicad_pcb (KiCad board)
At the start: 2 copper layers, 85 x 56 mm, 1 part, among them P1 CONN_13X2

Commit message: working on assigning footprints
Parts:
- added sot-89: Q***, 111kicad-jake:sot-89, F.Cu at (174.0, 151.1)
Changed lines of the file:
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@@
-(kicad_pcb (version 3) (host pcbnew "(2012-11-30 BZR 3829)-testing")
+(kicad_pcb (version 3) (host pcbnew "(2014-03-23 BZR 4768)-product")
   (general
     (links 0)
     (no_connects 0)
-    (area 127.606667 112.000001 242.964763 190.8)
+    (area 127.606667 112.000001 242.964763 187.88)
     (thickness 1.6)
     (drawings 41)
     (tracks 0)
     (zones 0)
-    (modules 1)
+    (modules 2)
     (nets 4)
   )
@@
       (usegerberextensions true)
       (excludeedgelayer true)
-      (linewidth 152400)
+      (linewidth 0.150000)
       (plotframeref false)
       (viasonmask false)
@@
     (uvia_dia 0.5)
     (uvia_drill 0.1)
-    (add_net "")
     (add_net +3.3V)
     (add_net +5V)
@@
     (fp_line (start -16.51 -2.54) (end -16.51 2.54) (layer F.SilkS) (width 0.2032))
     (fp_line (start 16.51 2.54) (end 16.51 -2.54) (layer F.SilkS) (width 0.2032))
-    (pad 1 thru_hole rect (at -15.24 1.27) (size 1.524 1.524) (drill 0.8128)
-      (layers *.Cu *.Mask F.SilkS)
-      (net 1 +3.3V)
-    )
-    (pad 2 thru_hole circle (at -15.24 -1.27) (size 1.524 1.524) (drill 1.016)
-      (layers *.Cu *.Mask F.SilkS)
-      (net 2 +5V)
-    )
-    (pad 3 thru_hole circle (at -12.7 1.27) (size 1.524 1.524) (drill 1.016)
-      (layers *.Cu *.Mask F.SilkS)
-    )
-    (pad 4 thru_hole circle (at -12.7 -1.27) (size 1.524 1.524) (drill 1.016)
-      (layers *.Cu *.Mask F.SilkS)
-    )
-    (pad 5 thru_hole circle (at -10.16 1.27) (size 1.524 1.524) (drill 1.016)
-      (layers *.Cu *.Mask F.SilkS)
-    )
-    (pad 6 thru_hole circle (at -10.16 -1.27) (size 1.524 1.524) (drill 1.016)
-      (layers *.Cu *.Mask F.SilkS)
-      (net 3 GND)
-    )
-    (pad 7 thru_hole circle (at -7.62 1.27) (size 1.524 1.524) (drill 1.016)
-      (layers *.Cu *.Mask F.SilkS)
-    )
-    (pad 8 thru_hole circle (at -7.62 -1.27) (size 1.524 1.524) (drill 1.016)
-      (layers *.Cu *.Mask F.SilkS)
-    )
-    (pad 9 thru_hole circle (at -5.08 1.27) (size 1.524 1.524) (drill 1.016)
-      (layers *.Cu *.Mask F.SilkS)
-    )
-    (pad 10 thru_hole circle (at -5.08 -1.27) (size 1.524 1.524) (drill 1.016)
-      (layers *.Cu *.Mask F.SilkS)
-    )
-    (pad 11 thru_hole circle (at -2.54 1.27) (size 1.524 1.524) (drill 1.016)
-      (layers *.Cu *.Mask F.SilkS)
-    )
-    (pad 12 thru_hole circle (at -2.54 -1.27) (size 1.524 1.524) (drill 1.016)
-      (layers *.Cu *.Mask F.SilkS)
-    )
-    (pad 13 thru_hole circle (at 0 1.27) (size 1.524 1.524) (drill 1.016)
-      (layers *.Cu *.Mask F.SilkS)
-    )
-    (pad 14 thru_hole circle (at 0 -1.27) (size 1.524 1.524) (drill 1.016)
-      (layers *.Cu *.Mask F.SilkS)
-    )
-    (pad 15 thru_hole circle (at 2.54 1.27) (size 1.524 1.524) (drill 1.016)
-      (layers *.Cu *.Mask F.SilkS)
-    )
-    (pad 16 thru_hole circle (at 2.54 -1.27) (size 1.524 1.524) (drill 1.016)
-      (layers *.Cu *.Mask F.SilkS)
-    )
-    (pad 17 thru_hole circle (at 5.08 1.27) (size 1.524 1.524) (drill 1.016)
-      (layers *.Cu *.Mask F.SilkS)
-    )
-    (pad 18 thru_hole circle (at 5.08 -1.27) (size 1.524 1.524) (drill 1.016)
-      (layers *.Cu *.Mask F.SilkS)
-    )
-    (pad 19 thru_hole circle (at 7.62 1.27) (size 1.524 1.524) (drill 1.016)
-      (layers *.Cu *.Mask F.SilkS)
-    )
-    (pad 20 thru_hole circle (at 7.62 -1.27) (size 1.524 1.524) (drill 1.016)
-      (layers *.Cu *.Mask F.SilkS)
-    )
-    (pad 21 thru_hole circle (at 10.16 1.27) (size 1.524 1.524) (drill 1.016)
-      (layers *.Cu *.Mask F.SilkS)
-    )
-    (pad 22 thru_hole circle (at 10.16 -1.27) (size 1.524 1.524) (drill 1.016)
-      (layers *.Cu *.Mask F.SilkS)
-    )
-    (pad 23 thru_hole circle (at 12.7 1.27) (size 1.524 1.524) (drill 1.016)
-      (layers *.Cu *.Mask F.SilkS)
-    )
-    (pad 24 thru_hole circle (at 12.7 -1.27) (size 1.524 1.524) (drill 1.016)
-      (layers *.Cu *.Mask F.SilkS)
-    )
-    (pad 25 thru_hole circle (at 15.24 1.27) (size 1.524 1.524) (drill 1.016)
-      (layers *.Cu *.Mask F.SilkS)
-    )
-    (pad 26 thru_hole circle (at 15.24 -1.27) (size 1.524 1.524) (drill 1.016)
-      (layers *.Cu *.Mask F.SilkS)
-    )
+    (pad 1 thru_hole rect (at -15.24 1.27) (size 1.524 1.524) (drill 0.8128) (layers *.Cu *.Mask F.SilkS)
+      (net 1 +3.3V))
+    (pad 2 thru_hole circle (at -15.24 -1.27) (size 1.524 1.524) (drill 1.016) (layers *.Cu *.Mask F.SilkS)
+      (net 2 +5V))
+    (pad 3 thru_hole circle (at -12.7 1.27) (size 1.524 1.524) (drill 1.016) (layers *.Cu *.Mask F.SilkS))
+    (pad 4 thru_hole circle (at -12.7 -1.27) (size 1.524 1.524) (drill 1.016) (layers *.Cu *.Mask F.SilkS))
+    (pad 5 thru_hole circle (at -10.16 1.27) (size 1.524 1.524) (drill 1.016) (layers *.Cu *.Mask F.SilkS))
+    (pad 6 thru_hole circle (at -10.16 -1.27) (size 1.524 1.524) (drill 1.016) (layers *.Cu *.Mask F.SilkS)
+      (net 3 GND))
+    (pad 7 thru_hole circle (at -7.62 1.27) (size 1.524 1.524) (drill 1.016) (layers *.Cu *.Mask F.SilkS))
+    (pad 8 thru_hole circle (at -7.62 -1.27) (size 1.524 1.524) (drill 1.016) (layers *.Cu *.Mask F.SilkS))
+    (pad 9 thru_hole circle (at -5.08 1.27) (size 1.524 1.524) (drill 1.016) (layers *.Cu *.Mask F.SilkS))
+    (pad 10 thru_hole circle (at -5.08 -1.27) (size 1.524 1.524) (drill 1.016) (layers *.Cu *.Mask F.SilkS))
+    (pad 11 thru_hole circle (at -2.54 1.27) (size 1.524 1.524) (drill 1.016) (layers *.Cu *.Mask F.SilkS))
+    (pad 12 thru_hole circle (at -2.54 -1.27) (size 1.524 1.524) (drill 1.016) (layers *.Cu *.Mask F.SilkS))
+    (pad 13 thru_hole circle (at 0 1.27) (size 1.524 1.524) (drill 1.016) (layers *.Cu *.Mask F.SilkS))
+    (pad 14 thru_hole circle (at 0 -1.27) (size 1.524 1.524) (drill 1.016) (layers *.Cu *.Mask F.SilkS))
+    (pad 15 thru_hole circle (at 2.54 1.27) (size 1.524 1.524) (drill 1.016) (layers *.Cu *.Mask F.SilkS))
+    (pad 16 thru_hole circle (at 2.54 -1.27) (size 1.524 1.524) (drill 1.016) (layers *.Cu *.Mask F.SilkS))
+    (pad 17 thru_hole circle (at 5.08 1.27) (size 1.524 1.524) (drill 1.016) (layers *.Cu *.Mask F.SilkS))
+    (pad 18 thru_hole circle (at 5.08 -1.27) (size 1.524 1.524) (drill 1.016) (layers *.Cu *.Mask F.SilkS))
+    (pad 19 thru_hole circle (at 7.62 1.27) (size 1.524 1.524) (drill 1.016) (layers *.Cu *.Mask F.SilkS))
+    (pad 20 thru_hole circle (at 7.62 -1.27) (size 1.524 1.524) (drill 1.016) (layers *.Cu *.Mask F.SilkS))
+    (pad 21 thru_hole circle (at 10.16 1.27) (size 1.524 1.524) (drill 1.016) (layers *.Cu *.Mask F.SilkS))
+    (pad 22 thru_hole circle (at 10.16 -1.27) (size 1.524 1.524) (drill 1.016) (layers *.Cu *.Mask F.SilkS))
+    (pad 23 thru_hole circle (at 12.7 1.27) (size 1.524 1.524) (drill 1.016) (layers *.Cu *.Mask F.SilkS))
+    (pad 24 thru_hole circle (at 12.7 -1.27) (size 1.524 1.524) (drill 1.016) (layers *.Cu *.Mask F.SilkS))
+    (pad 25 thru_hole circle (at 15.24 1.27) (size 1.524 1.524) (drill 1.016) (layers *.Cu *.Mask F.SilkS))
+    (pad 26 thru_hole circle (at 15.24 -1.27) (size 1.524 1.524) (drill 1.016) (layers *.Cu *.Mask F.SilkS))
     (model pin_array/pins_array_13x2.wrl
       (at (xyz 0 0 0))
       (scale (xyz 1 1 1))
+      (rotate (xyz 0 0 0))
+    )
+  )
+  (module 111kicad-jake:sot-89 (layer F.Cu)
+    (at 173.99 151.13)
+    (descr PowerMite3)
+    (attr smd)
+    (fp_text reference sot-89 (at 0.0508 -0.8382) (layer F.SilkS)
+      (effects (font (size 1.00076 1.00076) (thickness 0.20066)))
+    )
+    (fp_text value Q*** (at 0 1.0414) (layer F.SilkS) hide
+      (effects (font (size 1.00076 1.00076) (thickness 0.20066)))
+    )
+    (fp_line (start -0.889 -3.556) (end -0.889 -4.191) (layer F.SilkS) (width 0.127))
+    (fp_line (start -0.889 -4.191) (end 0.889 -4.191) (layer F.SilkS) (width 0.127))
+    (fp_line (start 0.889 -4.191) (end 0.889 -3.556) (layer F.SilkS) (width 0.127))
+    (fp_line (start -2.032 0.889) (end 2.032 0.889) (layer F.SilkS) (width 0.127))
+    (fp_line (start 2.032 0.889) (end 2.032 -3.556) (layer F.SilkS) (width 0.127))
+    (fp_line (start 2.032 -3.556) (end -2.032 -3.556) (layer F.SilkS) (width 0.127))
+    (fp_line (start -2.032 -3.556) (end -2.032 0.889) (layer F.SilkS) (width 0.127))
+    (fp_line (start 0.508 2.286) (end 1.397 2.286) (layer F.SilkS) (width 0.127))
+    (fp_line (start 1.397 2.286) (end 1.397 0.889) (layer F.SilkS) (width 0.127))
+    (fp_line (start 0.508 2.286) (end 0.508 0.889) (layer F.SilkS) (width 0.127))
+    (fp_line (start -1.397 2.286) (end -1.397 0.889) (layer F.SilkS) (width 0.127))
+    (fp_line (start -1.397 2.286) (end -0.508 2.286) (layer F.SilkS) (width 0.127))
+    (fp_line (start -0.508 2.286) (end -0.508 0.889) (layer F.SilkS) (width 0.127))
+    (pad 1 smd rect (at -0.9144 1.905) (size 0.9652 1.27) (layers F.Cu F.Paste F.Mask))
+    (pad 2 smd rect (at 0 -1.905) (size 4.826 5.334) (layers F.Cu F.Paste F.Mask))
+    (pad 3 smd rect (at 0.9144 1.905) (size 0.9652 1.27) (layers F.Cu F.Paste F.Mask))
+    (model smd/smd_transistors/powermite3.wrl
+      (at (xyz 0 0 0))
+      (scale (xyz 1 1 1))
