File: nukeanal.kicad_pcb (KiCad board)
At the start: 2 copper layers, 169.9 x 108.7 mm, 115 parts, among them P1 BNC, P2 CONN_1, P3 CONN_6, P4 CONN_2, P5 DE-9F, Q1 VN3205N8-G, Q2 MMBT5089, Q3 LP0701, Q4 MMBT5089, Q5 BSS83, Q6 BSS83, SW1 ONOFF, U1 OPA2365, U10 74HC14, U11 74HC74j, U2 MIC5209-3.3, U3 MIC5219YM5TR, U4 REF5045, U5 MIC5209-2.5, U6 OPA2365, U7 74HC14, U8 LM311N, U9 AD7983

Commit message: moved some caps around
Parts:
- moved CU6 82.2 mm to (185.5, 203.1), turned to 90 degrees
- moved CU5 79.6 mm to (183.4, 203.1), turned to 90 degrees
- moved CU7 52.6 mm to (180.2, 198.0)
- moved C17 52.0 mm to (180.2, 200.0)
- moved Q4 5.42 mm to (196.0, 182.8), turned to 0 degrees
Routing:
- net -0.25V: track 4.25 -> 24.7 mm, vias 0 -> 2
- net +5.25V: track 21.1 -> 40.4 mm
- net Net-(Q2-PadC): track 3.08 -> 17.7 mm
Changed lines of the file:
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@@
-(kicad_pcb (version 3) (host pcbnew "(2014-03-23 BZR 4768)-product")
+(kicad_pcb (version 3) (host pcbnew "(2014-05-31 BZR 4902)-product")
   (general
     (links 251)
-    (no_connects 213)
-    (area 127.434999 73.947599 297.505001 204.12644)
+    (no_connects 206)
+    (area 127.434999 73.947599 297.505001 205.100531)
     (thickness 1.6)
     (drawings 6)
-    (tracks 117)
+    (tracks 143)
     (zones 0)
     (modules 115)
@@
   )
   (setup
-    (last_trace_width 0.508)
+    (last_trace_width 0.2)
     (user_trace_width 0.254)
     (user_trace_width 0.508)
@@
       (plotreference true)
       (plotvalue true)
-      (plotothertext true)
       (plotinvisibletext false)
       (padsonsilk false)
@@
   )
   (module SMD_Packages:SM0805 placed (layer F.Cu)
-    (at 232.029 195.5165)
+    (at 180.213 200.025)
     (attr smd)
     (fp_text reference C17 (at 0 -0.3175) (layer F.SilkS)
@@
   )
   (module SMD_Packages:SM0805 placed (layer F.Cu)
-    (at 165.735 125.476)
+    (at 183.388 203.073 90)
     (attr smd)
-    (fp_text reference CU5 (at 0 -0.3175) (layer F.SilkS)
+    (fp_text reference CU5 (at 0 -0.3175 90) (layer F.SilkS)
       (effects (font (size 0.50038 0.50038) (thickness 0.10922)))
     )
-    (fp_text value 104 (at 0 0.381) (layer F.SilkS)
+    (fp_text value 104 (at 0 0.381 90) (layer F.SilkS)
       (effects (font (size 0.50038 0.50038) (thickness 0.10922)))
     )
@@
     (fp_line (start 1.524 -0.762) (end 1.524 0.762) (layer F.SilkS) (width 0.09906))
     (fp_line (start 1.524 0.762) (end 0.508 0.762) (layer F.SilkS) (width 0.09906))
-    (pad 1 smd rect (at -0.9525 0) (size 0.889 1.397) (layers F.Cu F.Paste F.Mask)
+    (pad 1 smd rect (at -0.9525 0 90) (size 0.889 1.397) (layers F.Cu F.Paste F.Mask)
       (net 5 GND))
-    (pad 2 smd rect (at 0.9525 0) (size 0.889 1.397) (layers F.Cu F.Paste F.Mask)
+    (pad 2 smd rect (at 0.9525 0 90) (size 0.889 1.397) (layers F.Cu F.Paste F.Mask)
       (net 16 +5.25V))
     (model smd/chip_cms.wrl
@@
   )
   (module SMD_Packages:SM0805 placed (layer F.Cu)
-    (at 165.735 123.2535)
+    (at 185.547 203.073 90)
     (attr smd)
-    (fp_text reference CU6 (at 0 -0.3175) (layer F.SilkS)
+    (fp_text reference CU6 (at 0 -0.3175 90) (layer F.SilkS)
       (effects (font (size 0.50038 0.50038) (thickness 0.10922)))
     )
-    (fp_text value 225 (at 0 0.381) (layer F.SilkS)
+    (fp_text value 225 (at 0 0.381 90) (layer F.SilkS)
       (effects (font (size 0.50038 0.50038) (thickness 0.10922)))
     )
@@
     (fp_line (start 1.524 -0.762) (end 1.524 0.762) (layer F.SilkS) (width 0.09906))
     (fp_line (start 1.524 0.762) (end 0.508 0.762) (layer F.SilkS) (width 0.09906))
-    (pad 1 smd rect (at -0.9525 0) (size 0.889 1.397) (layers F.Cu F.Paste F.Mask)
+    (pad 1 smd rect (at -0.9525 0 90) (size 0.889 1.397) (layers F.Cu F.Paste F.Mask)
       (net 5 GND))
-    (pad 2 smd rect (at 0.9525 0) (size 0.889 1.397) (layers F.Cu F.Paste F.Mask)
+    (pad 2 smd rect (at 0.9525 0 90) (size 0.889 1.397) (layers F.Cu F.Paste F.Mask)
       (net 16 +5.25V))
     (model smd/chip_cms.wrl
@@
   )
   (module SMD_Packages:SM0805 placed (layer F.Cu)
-    (at 232.029 189.23)
+    (at 180.213 197.993)
     (attr smd)
     (fp_text reference CU7 (at 0 -0.3175) (layer F.SilkS)
@@
   )
   (module Housings_SOT-23_SOT-143_TSOT-6:SOT23_Transistor_BC846_Handsoldering_RevB_14Mar2014 placed (layer F.Cu)
-    (at 192.8495 187.2615 180)
+    (at 196 182.85)
     (descr "SOT23,  Transistor, Handsoldering, BC846,")
     (tags "SOT23,  Transistor, Handsoldering, BC846,")
     (attr smd)
-    (fp_text reference Q4 (at -0.0005 3.5365 180) (layer F.SilkS)
+    (fp_text reference Q4 (at -0.0005 3.5365) (layer F.SilkS)
       (effects (font (thickness 0.3048)))
     )
-    (fp_text value MMBT5089 (at 0 3.81 180) (layer F.SilkS)
+    (fp_text value MMBT5089 (at 0 3.81) (layer F.SilkS)
       (effects (font (thickness 0.3048)))
     )
@@
     (fp_line (start 1.29916 -0.65024) (end 1.49982 -0.65024) (layer F.SilkS) (width 0.381))
     (fp_line (start 1.49982 -0.65024) (end 1.49982 0.0508) (layer F.SilkS) (width 0.381))
-    (pad B smd rect (at -0.95 1.50114 180) (size 0.8001 1.80086) (layers F.Cu F.Paste F.Mask)
+    (pad B smd rect (at -0.95 1.50114) (size 0.8001 1.80086) (layers F.Cu F.Paste F.Mask)
       (net 76 "Net-(Q4-PadB)"))
-    (pad E smd rect (at 0.95 1.50114 180) (size 0.8001 1.80086) (layers F.Cu F.Paste F.Mask)
+    (pad E smd rect (at 0.95 1.50114) (size 0.8001 1.80086) (layers F.Cu F.Paste F.Mask)
       (net 5 GND))
-    (pad C smd rect (at 0 -1.50114 180) (size 0.8001 1.80086) (layers F.Cu F.Paste F.Mask)
+    (pad C smd rect (at 0 -1.50114) (size 0.8001 1.80086) (layers F.Cu F.Paste F.Mask)
       (net 77 "Net-(Q4-PadC)"))
   )
@@
   (segment (start 171.775 195.3895) (end 172.067 195.3895) (width 0.508) (layer F.Cu) (net 16))
   (segment (start 172.067 195.3895) (end 174.425 196.2725) (width 0.508) (layer F.Cu) (net 16) (status 20))
-  (segment (start 189.738 196.596) (end 187.554 196.596) (width 0.508) (layer F.Cu) (net 16))
-  (segment (start 187.05 197.1) (end 187.05 201.85) (width 0.508) (layer F.Cu) (net 16))
-  (segment (start 187.554 196.596) (end 187.05 197.1) (width 0.508) (layer F.Cu) (net 16))
   (segment (start 166.9295 195.3895) (end 171.3 195.3895) (width 0.508) (layer F.Cu) (net 16))
   (segment (start 171.3 195.3895) (end 171.323 195.3895) (width 0.508) (layer F.Cu) (net 16))
   (segment (start 164.495 191.746) (end 164.495 192.955) (width 0.508) (layer F.Cu) (net 16))
   (segment (start 164.495 192.955) (end 166.9295 195.3895) (width 0.508) (layer F.Cu) (net 16))
+  (segment (start 187.554 196.596) (end 187.05 197.1) (width 0.508) (layer F.Cu) (net 16))
+  (segment (start 187.05 201.803) (end 187.05 201.85) (width 0.508) (layer F.Cu) (net 16))
+  (segment (start 187.05 197.1) (end 187.05 201.803) (width 0.508) (layer F.Cu) (net 16))
+  (segment (start 187.554 196.596) (end 189.738 196.596) (width 0.508) (layer F.Cu) (net 16))
+  (segment (start 186.7325 202.1205) (end 187.05 201.803) (width 0.508) (layer F.Cu) (net 16))
+  (segment (start 185.547 202.1205) (end 186.7325 202.1205) (width 0.508) (layer F.Cu) (net 16))
+  (segment (start 177.2725 196.2725) (end 176.497 200.277) (width 0.508) (layer F.Cu) (net 16))
+  (segment (start 176.497 200.277) (end 176.497 201.827) (width 0.508) (layer F.Cu) (net 16))
+  (segment (start 176.497 201.827) (end 181.3 201.85) (width 0.508) (layer F.Cu) (net 16))
+  (segment (start 174.425 196.2725) (end 177.2725 196.2725) (width 0.508) (layer F.Cu) (net 16))
+  (segment (start 181.5705 202.1205) (end 181.3 201.85) (width 0.508) (layer F.Cu) (net 16))
+  (segment (start 183.388 202.1205) (end 181.5705 202.1205) (width 0.508) (layer F.Cu) (net 16))
+  (segment (start 185.547 202.1205) (end 183.388 202.1205) (width 0.508) (layer F.Cu) (net 16))
   (segment (start 168.4475 199.475) (end 168.305 199.3325) (width 0.508) (layer F.Cu) (net 19))
   (segment (start 168.305 199.3325) (end 168.305 197.334) (width 0.508) (layer F.Cu) (net 19))
   (segment (start 168.4475 199.475) (end 168.4475 201.525) (width 0.508) (layer F.Cu) (net 19) (status 20))
+  (segment (start 182.356 200.406) (end 182.35 200.4) (width 0.508) (layer F.Cu) (net 19))
+  (via (at 182.35 200.4) (size 0.9) (layers F.Cu B.Cu) (net 19))
+  (segment (start 182.35 200.4) (end 179.425 197.475) (width 0.508) (layer B.Cu) (net 19))
+  (segment (start 179.425 197.475) (end 169.95 197.475) (width 0.508) (layer B.Cu) (net 19))
+  (via (at 169.95 197.475) (size 0.9) (layers F.Cu B.Cu) (net 19))
+  (segment (start 169.95 197.475) (end 169.809 197.334) (width 0.508) (layer F.Cu) (net 19))
+  (segment (start 169.809 197.334) (end 168.305 197.334) (width 0.508) (layer F.Cu) (net 19))
+  (segment (start 184.15 200.406) (end 182.356 200.406) (width 0.508) (layer F.Cu) (net 19))
+  (segment (start 181.1655 200.025) (end 181.1655 197.993) (width 0.508) (layer F.Cu) (net 19))
+  (segment (start 181.5405 200.4) (end 181.1655 200.025) (width 0.508) (layer F.Cu) (net 19))
+  (segment (start 182.35 200.4) (end 181.5405 200.4) (width 0.508) (layer F.Cu) (net 19))
   (segment (start 191.60448 192.9495) (end 191.7065 193.05152) (width 0.508) (layer F.Cu) (net 23))
   (segment (start 191.7065 193.05152) (end 191.7065 195.74002) (width 0.762) (layer F.Cu) (net 23))
@@
   (segment (start 179.0065 189.32652) (end 179.0065 188.76264) (width 0.508) (layer F.Cu) (net 75))
   (segment (start 177.2285 191.10452) (end 179.0065 189.32652) (width 0.508) (layer F.Cu) (net 75))
+  (segment (start 179.80452 191.10452) (end 182.475 191.2) (width 0.508) (layer F.Cu) (net 75))
+  (segment (start 182.475 191.2) (end 182.475 196.975) (width 0.508) (layer F.Cu) (net 75))
+  (segment (start 182.475 196.975) (end 182.753 199.136) (width 0.508) (layer F.Cu) (net 75))
+  (segment (start 182.753 199.136) (end 184.15 199.136) (width 0.508) (layer F.Cu) (net 75))
+  (segment (start 177.2285 191.10452) (end 179.80452 191.10452) (width 0.508) (layer F.Cu) (net 75))
   (segment (start 189.76848 184.11952) (end 190.0555 183.8325) (width 0.508) (layer F.Cu) (net 76))
   (segment (start 190.0555 183.8325) (end 193.167 183.8325) (width 0.508) (layer F.Cu) (net 76))
   (segment (start 193.167 183.8325) (end 193.7995 184.465) (width 0.508) (layer F.Cu) (net 76))
-  (segment (start 193.7995 184.465) (end 193.7995 185.76036) (width 0.508) (layer F.Cu) (net 76))
+  (segment (start 193.7995 184.465) (end 195.05 184.35114) (width 0.508) (layer F.Cu) (net 76) (status 20))
   (segment (start 189.76848 185.547) (end 189.76848 184.11952) (width 0.508) (layer F.Cu) (net 76))
 )
