File: nukeanal.sch (KiCad schematic (older format))
At the start: 83 parts, among them P1 CONN_2, P2 CONN_2, P3 CONN_2, Q1 VN3205, Q2 MMBT5089, Q3 LP0701, Q4 MMBT5089, Q5 FET_N, Q6 FET_N, SW1 ONOFF, U1 LM358, U10 74HC14, U11 74HC74, U2 LE33CD, U4 REF5045, U5 MIC5209-2.5, U6 LM358, U7 74HC14, U8 LM311N, U9 AD7983

Commit message: working on assigning footprints
Parts:
- removed U?: LE50CD, symbol LE33-SO8
- added U3: MIC5219YM5TR, symbol MIC5219YM5TR
- C1, C2: value wesfdsdfds -> 100; footprint (none) -> SMD_Packages:SM0805
- C10, C4, C7, C9, R28: footprint (none) -> SMD_Packages:SM0805
- C3, C5, C6, CU4: footprint (none) -> SMD_Packages:SM1206
- C8: footprint (none) -> SMD_Packages:SM1206POL
- D1, D2: footprint (none) -> SMD_Packages:SM1210L
- D3, D4: value DIODE -> DPAD1
- Q1: value VN3205 -> VN3205N8-G; footprint (none) -> ~
- Q5, Q6: footprint BSS_83 -> (none)
- R11: value 5K -> 422705
- R12: value 150 -> 100K
- U1, U6: value LM358 -> OPA2365
- U5: footprint (none) -> sot223
Connections:
- net labels added: +5.25V, -0.25V
- net labels removed: -0.35V
- wire segments 114 -> 118
Other:
- note added: "Vee"
- note added: "change to 5.25v Vdd and -0.25v Vee"
- moved on the sheet: C1, C10, C2, C3, C4, C5, C6, C7, C8, C9, CU4, D1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

Commit message: finished with schematic, footprint assignment, but no board yet
Parts:
- removed C8: 226, SMD_Packages:SM1206POL, symbol C
- removed D3, D4: DPAD1, symbol DIODE
- removed P1, P2: CONN_2, symbol CONN_2
- removed Q5, Q6: FET_N, symbol FET_N
- added C11: 104, SMD_Packages:SM0805, symbol C
- added C12: 225, SMD_Packages:SM0805, symbol C
- added C8: 226, Capacitors:CP_5x6mm, symbol CAPAPOL
- added D3: DPAD1, 222TO-78:TO-78_Housing_5Pin, symbol DPAD1
- added K1: CONN_3, Connect:SIL-3, symbol CONN_3
- added P1: BNC, 111kicad-jake:bnc-rocket, symbol BNC
- added Q5, Q6: BSS83, Transistors_SMD:sot143B, symbol BSS83
- C3, C5: footprint SMD_Packages:SM1206 -> SMD_Packages:SM0805
- C6: footprint SMD_Packages:SM1206 -> Capacitors_ThroughHole:Capacitor13x4RM10
- CU4: value 105 -> 225; footprint SMD_Packages:SM1206 -> SMD_Packages:SM0805
- D1, D2: footprint SMD_Packages:SM1210L -> Diodes_ThroughHole:Diode_DO-41_SOD81_Horizontal_RM10
- D10, D11, D12, D13, D14, D8, D9: value DIODE -> 1N4148; footprint (none) -> Diodes_ThroughHole:Diode_DO-35_SOD27_Horizontal_RM10
- D5: footprint (none) -> Diodes_ThroughHole:Diode_DO-35_SOD27_Horizontal_RM10
- D6, D7: footprint (none) -> Diodes_ThroughHole:Diode_DO-41_SOD81_Horizontal_RM10
- P4: renamed from P3; footprint (none) -> Connect:bornier2
- Q1: footprint ~ -> Discret:TO92DGS
- Q2, Q4: footprint (none) -> Housings_SOT-23_SOT-143_TSOT-6:SOT23_Transistor_BC846_Handsoldering_RevB_14Mar2014
- Q3: footprint (none) -> Discret:TO92DGS
- R1, R10, R11, R12, R13, R14, R16, R17, R19, R2, R20, R21, R22, R23, R24, R25, R26, R27, R29, R3, R30, R31, R32, R33, R34, R35, R36, R37, R4, R5, R6, R7, R8: footprint (none) -> Resistors_SMD:Resistor_SMD0805_HandSoldering
- R15, R18, R9: footprint (none) -> Resistors_ThroughHole:Resistor_Horizontal_RM10mm
- R28: footprint SMD_Packages:SM0805 -> Resistors_SMD:Resistor_SMD0805_HandSoldering
- SW1: footprint (none) -> Pin_Headers:Pin_Header_Straight_1x02
- U1, U2, U4, U6, U8: footprint (none) -> Power_Integrations:SO-8
- U10, U11, U7: footprint (none) -> SMD_Packages:SO14N
- U3: footprint (none) -> SMD_Packages:SOT23-5
- U5: footprint sot223 -> 111kicad-jake:SOT-223-3
- U9: footprint (none) -> SMD_Packages:MSOP10-0.5
Connections:
- net +3.3V: now also U2.1 (VO)
- net BATT+: now also U2.8 (VI)
- net GND: now also C10.1, C3.1, C8.2, P1.2 (Ext), Q5.2 (S), Q6.2 (S); no longer C10.2, C3.2
- net REF45: now also C8.1
- net at R29.2, R30.2, U7.10: now also Q5.4 (G)
- net at R30.1, U10.9: now also C10.2; no longer C10.1
- net at D13.1 (A), R31.2, U10.12: now also Q6.4 (G)
- net at R25.2, R26.2: now also Q5.3 (D), Q6.3 (D)
- net at U6.6 (-), U6.7, U9.3 (+IN): now also R17.1; no longer R17.2
- net at R20.1: now also D3.5 (K)
- net at C4.2, U6.1: now also D3.1 (K), D3.7 (A)
- net at R13.2, U6.2 (-): now also R17.2, D3.2 (A); no longer R17.1
- net at R1.2: now also K1.3 (P3)
- net at R2.2: now also K1.1 (P1)
- net at U4.5 (TRIM/NR): now also C3.2
- net at U4.7 (NC): no longer C3.1
- new net: K1.2 (PM), P1.1 (In)
Other:
- moved on the sheet: C10, C3, R17, R20, R25, R29, R31

Commit message: merge from .zip download of jerry's latest commit
Parts:
- removed Q2, Q4: MMBT5089, Housings_SOT-23_SOT-143_TSOT-6:SOT23_Transistor_BC846_Handsoldering_RevB_14Mar2014, symbol 2SC1941
- removed U11: 74HC74, SMD_Packages:SO14N, symbol 74HC74
- removed U2: LE33CD, Power_Integrations:SO-8, symbol LE33-SO8
- removed U5: MIC5209-2.5, 111kicad-jake:SOT-223-3, symbol 7805
- added C13, C15, C16, C17, C19, C21, C23, C25, C27, C29, C31, C33, CU2, CU6: 225, SMD_Packages:SM0805, symbol C
- added C14, C18, C20, C22, C24, C26, C28, C30, C32, CU1, CU3, CU41, CU5, CU7: 104, SMD_Packages:SM0805, symbol C
- added P2: CONN_1, 111kicad-jerry:testpin037, symbol CONN_1
- added P3: CONN_6, 111kicad-jerry:6x1pin037, symbol CONN_6
- added P5: DE-9F, 111kicad-jerry:DB9FC, symbol CONN_9
- added Q2, Q4: MMBT5089, symbol MMBT5089
- added U11: 74HC74j, SMD_Packages:SO14N, symbol 74HC74j
- added U2: MIC5209-3.3, symbol MIC5209
- added U5: MIC5209-2.5, symbol MIC5209
Connections:
- net +5.15V is gone; now on net +5.25V: CU4.1, U4.2 (VIN)
- net +2.5V: now also C24.2, C25.2, C30.2, C31.2, U5.3 (VO)
- net +3.3V: now also C18.2, C19.2, C20.2, C21.2, C22.2, C23.2, C26.2, C27.2, C32.2, C33.2, U11.1 (Cd), U11.14 (VCC), U11.2 (D), U11.3 (Cp), U11.4 (Sd), U2.3 (VO)
- net +5.25V: now also C11.2, C13.2, C28.2, C29.2, CU1.2, CU2.2, CU41.2, CU5.2, CU6.2, U5.1 (VI)
- net -0.25V: now also C16.2, C17.2, CU3.2, CU7.2
- net -0.5V: now also C14.2, C15.2
- net BATT+: now also U2.1 (VI); no longer U3.1 (VIN)
- net GND: now also C11.1, C12.1, C13.1, C14.1, C15.1, C16.1, C17.1, C18.1, C19.1, C20.1, C21.1, C22.1, C23.1, C24.1, C25.1, C26.1, C27.1, C28.1, C29.1, C30.1, C31.1, C32.1, C33.1, CU1.1, CU2.1, CU3.1, CU41.1, CU5.1, CU6.1, CU7.1, P3.1, P3.2, P5.1 (P1), P5.2 (P2), P5.3 (P3), P5.4 (P4), P5.5 (P5), Q2.E, Q4.E, U11.12 (D), U11.7 (GND), U2.2 (GND), U5.2 (GND)
- net SCLK: now also P3.4, P5.7 (P7)
- net SDO: now also P3.3, P5.6 (P6)
- net TEST: now also P2.1, U11.13 (Cd)
- net ~CE: now also P3.5, P5.8 (P8)
- net ~REQ: now also P3.6, P5.9 (P9)
- net at U10.10: now also U11.11 (Cp)
- net at D14.1 (A), R36.2, R37.2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: now also U11.10 (Sd)
- net at D11.1 (A): now also U11.8 (~Q)
- net at D12.1 (A), R35.2: now also U11.9 (Q)
- net at R10.1, U6.3 (+), U8.3 (-): now also Q2.C
- net at R21.1: now also Q4.C
- net at R19.1: now also Q4.B
- net at R14.2: now also Q2.B
- net at R11.2, R12.2, U3.4 (ADJ): now also C12.2
Other:
- note added: "for U1"
- note added: "for U10"
- note added: "for U11"
- note added: "for U6"
- note added: "for U7"
- note added: "for U8"
- note added: "for U9"
- note added: "for reg"
- note removed: "change to 5.25v Vdd and -0.25v Vee"
- moved on the sheet: C12
